Commit message: ridgebackgazebo_working

File: ridgeback_yumi/ridgeback_yumi_description/urdf/ridgeback_yumi.urdf.xacro (robot description, xacro)
@@ -13,23 +13,30 @@
   <xacro:include filename="$(find yumi_description)/urdf/Extras/yumi_optodaq_sensors.xacro"/-->
   <!-- Import Gazebo plugins -->
-  <xacro:include filename="$(find yumi_description)/urdf/Gazebo/gazebo.urdf.xacro"/>
+  <xacro:include filename="$(find yumi_description)/urdf/Gazebo/gazebo.urdf.xacro"/> <!--THIS IS THE CULPRIT - LOADS GAZEBO_ROS_CONTROL TWICE-->
   <!--yumi-->
   <xacro:yumi name="yumi" hardware_interface="hardware_interface/VelocityJointInterface" parent="yumi_pedestal">
     <origin xyz="0 0 0.1" rpy="0 0 0" />
   </xacro:yumi>
-  <!--xacro:yumi_optodaq_sensor name="optodaq_r" parent="yumi_link_7_r">
+  <!--optodaq
+  <xacro:yumi_optodaq_sensor name="optodaq_r" parent="yumi_link_7_r">
       <origin xyz="0 0 0.033" rpy="0 ${PI} ${-PI/4}" />
   </xacro:yumi_optodaq_sensor>
   <xacro:yumi_optodaq_sensor name="optodaq_l" parent="yumi_link_7_l">
 	  <origin xyz="0 0 0.033" rpy="0 ${PI} ${-PI/4}" />
-  </xacro:yumi_optodaq_sensor>
-  <right gripper
+  </xacro:yumi_optodaq_sensor
   <xacro:yumi_servo_gripper name="gripper_r" hardware_interface="hardware_interface/EffortJointInterface" parent="optodaq_r_sensor_link">
     <origin xyz="0 0 -0.033" rpy="${PI} 0.0 ${PI/4}" />
   </xacro:yumi_servo_gripper>
-  <left gripper-
   <xacro:yumi_servo_gripper name="gripper_l" hardware_interface="hardware_interface/EffortJointInterface" parent="optodaq_l_sensor_link">
     <origin xyz="0 0 -0.033" rpy="${PI} 0.0 ${PI/4}" />
   </xacro:yumi_servo_gripper-->
+  <!--right gripper-->
+  <xacro:yumi_servo_gripper name="gripper_r" hardware_interface="hardware_interface/EffortJointInterface" parent="yumi_link_7_r">
+    <origin xyz="0 0 0.007" rpy="0 0 ${PI}" />
+  </xacro:yumi_servo_gripper>
+  <!--left gripper-->
+  <xacro:yumi_servo_gripper name="gripper_l" hardware_interface="hardware_interface/EffortJointInterface" parent="yumi_link_7_l">
+    <origin xyz="0 0 0.007" rpy="0 0 ${PI}" />
+  </xacro:yumi_servo_gripper>
   <xacro:property name="pedestal_height" value="0.28" />
   <xacro:property name="pedestal_offset_x" value="0.32" />
@@ -64,4 +71,5 @@
     <child link="yumi_base_link" />
   </joint>
+ <!--kinect
   <link name="kinect2">
     <visual>
@@ -69,5 +77,5 @@
       <geometry>
                     <box size="0.4 0.02 0.02" />
-        <!--mesh scale="0.001 0.001 0.001" filename="package://yumi_description/meshes/accesories/KinectXboxOne.stl"/-->
+        <mesh scale="0.001 0.001 0.001" filename="package://yumi_description/meshes/accesories/KinectXboxOne.stl"/>
       </geometry>
       <material name="Black" />
@@ -120,4 +128,4 @@
     <child link="kinect2" />
     <origin rpy="${-PI/2} 0 ${kinect_zrotation_fix}" xyz="0.25 0 0" />
-  </joint>
+  </joint-->
 </robot>
