Commit message: ridgebackgazebo_turtlebot

File: ridgeback_yumi/ridgeback_yumi_description/urdf/ridgeback_yumi.urdf (robot description, URDF)
Before this commit: robot ridgeback_yumi, 48 links, 47 joints
Links:
- removed link kinect2
- removed link left_kinect_base
- removed link middle_kinect_base
- removed link right_kinect_base
Joints:
- removed joint kinect2_to_left_kinect_base
- removed joint kinect2_to_right_kinect_base
- removed joint middle_kinect_base_to_kinect2
- removed joint yumi_to_middle_kinect_base
